File: Schematics/Weapons/Weapons panel.sch (EAGLE design)
At the start: 63 parts, among them T1 2n2222, T2 2n2222, T3 2n2222, T4 2n2222, U1 ATMEGA328P, Y1 16MHz

Commit message: Updated weapons panel schematic
Parts:
- removed JP2: FTDI, SparkFun-Connectors:ARDUINO_SERIAL_PROGRAMPTH
- removed U1: ATMEGA328P, SparkFun-DigitalIC:ATMEGA328_SMT
- removed Y1: 16MHz, SparkFun-FreqCtrl:RESONATOR16MHZ
- added CN1: (no value), adafruit:DCBARRELPTH
- added LED25: Reload 1, adafruit:LED5MM
- added LED26: Reload 2, adafruit:LED5MM
- added LED27: Fire 1, adafruit:LED5MM
- added LED28: Fire 2, adafruit:LED5MM
- added LED29: Charging 1, adafruit:LED5MM
- added LED30: Charging 2, adafruit:LED5MM
- added LED31: Acquired, adafruit:LED5MM
- added R30, R31, R32, R33, R34, R35: (no value), resistor:R-US_0204/7
- added S10, S5: Fire 2, adafruit:SPST
- added S11: Left, adafruit:SPST
- added S12: Right, adafruit:SPST
- added S13: Lock, adafruit:SPST
- added S3, S8: Arm, SparkFun-Electromechanical:SWITCH-SPDTPTH
- added S4, S9: Fire 1, adafruit:SPST
- added S6: Reload 1, adafruit:SPST
- added S7: Reload 2, adafruit:SPST
- added U$3: MODULATION, circular_led_breakout:CIRCULAR_LED_BREAKOUT
- R29: value 10k -> (none); device SparkFun-Passives:RESISTORKIT -> resistor:R-US_0204/7
- U$1: value FREQUENCY -> ARDUINO-TEENSY++; device circular_led_breakout:CIRCULAR_LED_BREAKOUT -> teensypp:ARDUINO-TEENSY++
- U$2: value MODULATION -> FREQUENCY
Connections:
- removed net N$40: U1.PB6(XTAL1/TOSC1), Y1.1
- removed net RXD: JP2.TXO, U1.PD0(RXD)
- removed net TXD: JP2.RXI, U1.PD1(TXD)
- new net ENC1_G: U$1.17, U$2.GRN
- new net ENC1_R: U$1.15,PWM, U$2.RED
- new net ENC2_G: U$1.10, U$3.GRN
- new net ENC2_R: U$1.16,PWM, U$3.RED
- new net L0: S8.P, U$1.29
- new net L1: S9.P, U$1.30
- new net L2: S10.P, U$1.31
- new net L3: R31.2, U$1.32
- new net L4: R32.2, U$1.33
- new net L5: R33.2, U$1.34
- new net L6: R34.2, U$1.35
- new net N$33: LED25.A, R29.1
- new net N$34: LED26.A, R30.1
- new net N$35: LED27.A, R31.1
- new net N$36: LED28.A, R32.1
- new net N$37: LED29.A, R33.1
- new net T0: S3.P, U$1.40,A2
- new net T1: S4.P, U$1.41,A3
- new net T2: S5.P, U$1.42,A4
- new net T3: S6.P, U$1.43,A5
- new net T4: S7.P, U$1.44,A6
- new net T5: R29.2, U$1.45,A7
- new net T6: R30.2, U$1.28
- new net TS_0: S11.S, U$1.11
- new net TS_1: S12.S, U$1.12
- new net TS_2: S13.S, U$1.13
- new net TS_3: R35.1, U$1.14,PWM
- net 5V: now also CN1.PWR, S3.O, S8.O, U$3.VCC; no longer JP2.VCC, R29.2, U1.AREF, U1.AVCC, U1.VCC@1, U1.VCC@2
- net BOTTOM: now also U$1.27,PWM; no longer U1.PC3(ADC3)
- net CLK: now also U$1.21, U$3.CLK; no longer U$1.CLK, U1.PB3(MOSI/OC2)
- net CLR: now also U$1.23, U$3.CLR; no longer U$1.CLR, U1.PB2(SS/OC1B)
- net DAT: now also U$1.22, U$3.DAT; no longer U$1.DAT, U1.PB0(ICP)
- net EN: now also U$1.20, U$3.EN; no longer U$1.EN, U1.PB5(SCK)
- net ENC1_A: now also U$1.18,INT6, U$2.A; no longer U$1.A, U1.PD3(INT1)
- net ENC1_B: now also U$1.19, U$2.B; no longer U$1.B, U1.PD2(INT0)
- net ENC2_A: now also U$1.36,INT4, U$3.A; no longer U$2.A, U1.PD5(T1)
- net ENC2_B: now also U$1.37,INT5, U$3.B; no longer U$2.B, U1.PD4(XCK/T0)
- net GND: now also CN1.GND, LED25.C, LED26.C, LED27.C, LED28.C, LED29.C, LED30.C, LED31.C, S10.S, S11.P, S12.P, S13.P, S3.S, S4.S, S5.S, S6.S, S7.S, S8.S, S9.S, U$3.GND; no longer JP2.CTS, JP2.GND, U1.AGND, U1.GND@1, U1.GND@2, Y1.2
- net LATCH1: now also U$1.38,A0, U$2.LATCH; no longer U$1.LATCH, U1.PD6(AIN0)
- net LATCH2: now also U$1.39,A1, U$3.LATCH; no longer U$2.LATCH, U1.PD7(AIN1)
- net LEFT: now also U$1.26,PWM; no longer U1.PC0(ADC0)
- net N$38: now also LED30.A, R34.1; no longer JP2.DTR, R29.1, U1.PC6(/RESET)
- net N$39: now also LED31.A, R35.2; no longer U1.PB7(XTAL2/TOSC2), Y1.3
- net RIGHT: now also U$1.24,PWM; no longer U1.PC2(ADC2)
- net SCL: now also U$1.0,PWM,INT0; no longer U1.PC5(ADC5/SCL)
- net SDA: now also U$1.1,PWM,INT1; no longer U1.PC4(ADC4/SDA)
- net TOP: now also U$1.25,PWM; no longer U1.PC1(ADC1)
Other:
- note added: "Frequency"
- note added: "I2C"
- note added: "Lasers"
- note added: "Modulation"
- note added: "Power in"
- note added: "Shields"
- note added: "Targeting System"
- note added: "Torpedos"
- moved on the sheet: JP1, LED1, LED10, LED11, LED12, LED13, LED14, LED15, LED16, LED17, LED18, LED19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
